File: AstraControlPowerPCB/AstraControlPower.kicad_pcb (KiCad board)
At the start: 4 copper layers, 40 x 60 mm, 1 part, among them CN1 WJ124_5P

Commit message: Finished layout
Parts:
- added CN2: WJ124_5P, LiveAstra:CN_SCREW_TERMINAL_WJ124_4P-P3.81_KF124-4P, F.Cu at (170.0, 126.0)
- added CN3: WJ124_5P, LiveAstra:CN_SCREW_TERMINAL_WJ124_4P-P3.81_KF124-4P, F.Cu at (170.0, 94.0)
- added CN4: WJ124_5P, LiveAstra:CN_SCREW_TERMINAL_WJ124_4P-P3.81_KF124-4P, F.Cu at (150.0, 94.0)
- added CN5: WJ124_5P, LiveAstra:CN_SCREW_TERMINAL_WJ124_4P-P3.81_KF124-4P, F.Cu at (150.0, 126.0)
- added CN6: WJ124_5P, LiveAstra:CN_SCREW_TERMINAL_WJ124_5P-P3.81_KF124-5P, F.Cu at (166.0, 110.0)
- added JP1: JP_SolderJumper_2_Bridged, Jumper:SolderJumper-2_P1.3mm_Bridged_RoundedPad1.0x1.5mm, B.Cu at (165.0, 130.2)
- CN1: footprint LiveAstra:CN_SCREW_TERMINAL_WJ124_5P-P3.81_KF124-3.81-5P -> LiveAstra:CN_SCREW_TERMINAL_WJ124_5P-P3.81_KF124-5P
- moved CN1 10.8 mm to (154.0, 110.0), turned to 90 degrees
Connections:
- CN1 pad 1: unconnected-(CN1-Pin_1-Pad1) -> /Block Diagram/5V
- CN1 pad 2: unconnected-(CN1-Pin_2-Pad2) -> /Block Diagram/VIN
- CN1 pad 3: unconnected-(CN1-Pin_3-Pad3) -> GND
- CN1 pad 4: unconnected-(CN1-Pin_4-Pad4) -> /Block Diagram/RS485+
- CN1 pad 5: unconnected-(CN1-Pin_5-Pad5) -> /Block Diagram/RS485-
Routing:
- net /Block Diagram/RS485+: track 0.00 -> 28.0 mm
- net /Block Diagram/RS485-: track 0.00 -> 28.0 mm
- net /Block Diagram/VIN: track 0.00 -> 24.9 mm
- net /Block Diagram/5V: track 0.00 -> 20.6 mm
- net /Block Diagram/LED: track 0.00 -> 4.51 mm
- added copper zone on In2.Cu, net /Block Diagram/5V
- added copper zone on F.Cu, net /Block Diagram/VIN
- added copper zone on B.Cu, net /Block Diagram/VIN_SW
- added copper zone on B.Cu, net GND
- added copper zone on F.Cu, net GND
- added copper zone on In1.Cu, net GND
Other:
- board size 40 x 60 mm -> 40 x 44 mm

Commit message: Minor updates
Parts:
- added kibuzzard-676F3984: G***, kibuzzard-676F3984, F.Cu at (176.0, 130.8)
- added kibuzzard-676F399B: G***, kibuzzard-676F399B, F.Cu at (172.0, 130.8)
- added kibuzzard-676F39A3: G***, kibuzzard-676F39A3, F.Cu at (168.2, 130.8)
- added kibuzzard-676F39A3: G***, kibuzzard-676F39A3, F.Cu at (148.0, 130.8)
- added kibuzzard-676F39AF: G***, kibuzzard-676F39AF, F.Cu at (164.2, 130.8)
- added kibuzzard-676F39FE: G***, kibuzzard-676F39FE, F.Cu at (148.8, 117.8)
- added kibuzzard-676F39FE: G***, kibuzzard-676F39FE, F.Cu at (156.0, 130.8)
- added kibuzzard-676F3A03: G***, kibuzzard-676F3A03, F.Cu at (148.8, 110.0)
- added kibuzzard-676F3A03: G***, kibuzzard-676F3A03, F.Cu at (152.0, 130.8)
- added kibuzzard-676F3A03: G***, kibuzzard-676F3A03, F.Cu at (171.2, 110.0)
- added kibuzzard-676F3A07: G***, kibuzzard-676F3A07, F.Cu at (144.0, 130.8)
- added kibuzzard-676F3A8C: G***, kibuzzard-676F3A8C, F.Cu at (148.8, 114.0)
- added kibuzzard-676F3AEB: G***, kibuzzard-676F3AEB, F.Cu at (148.8, 102.5)
- added kibuzzard-676F3AEF: G***, kibuzzard-676F3AEF, F.Cu at (148.8, 106.2)
- added kibuzzard-676F3AFB: G***, kibuzzard-676F3AFB, F.Cu at (171.2, 106.2)
- added kibuzzard-676F3AFF: G***, kibuzzard-676F3AFF, F.Cu at (171.2, 113.8)
- added kibuzzard-676F3D01: G***, kibuzzard-676F3D01, F.Cu at (171.2, 118.1)
- added kibuzzard-676F3D0A: G***, kibuzzard-676F3D0A, F.Cu at (171.2, 102.2)
- added kibuzzard-676F3DF6: G***, kibuzzard-676F3DF6, F.Cu at (144.2, 89.2)
- added kibuzzard-676F3E04: G***, kibuzzard-676F3E04, F.Cu at (148.0, 89.2)
- added kibuzzard-676F3E0A: G***, kibuzzard-676F3E0A, F.Cu at (151.8, 89.2)
- added kibuzzard-676F3E29: G***, kibuzzard-676F3E29, F.Cu at (155.8, 89.2)
- added kibuzzard-676F3E9C: G***, kibuzzard-676F3E9C, F.Cu at (175.8, 89.2)
- added kibuzzard-676F3EA0: G***, kibuzzard-676F3EA0, F.Cu at (172.0, 89.2)
- added kibuzzard-676F3EA4: G***, kibuzzard-676F3EA4, F.Cu at (168.0, 89.2)
- added kibuzzard-676F3EA7: G***, kibuzzard-676F3EA7, F.Cu at (164.2, 89.2)
- added kibuzzard-676F3F6C: G***, kibuzzard-676F3F6C, F.Cu at (176.0, 116.2)
- added kibuzzard-676F3F74: G***, kibuzzard-676F3F74, F.Cu at (144.0, 116.2)
- added kibuzzard-676F3FB0: G***, kibuzzard-676F3FB0, F.Cu at (144.0, 120.5)
- added kibuzzard-676F3FBD: G***, kibuzzard-676F3FBD, F.Cu at (174.2, 120.5)
- added kibuzzard-676F4051: G***, kibuzzard-676F4051, F.Cu at (160.0, 110.0)
- added kibuzzard-676F4065: G***, kibuzzard-676F4065, F.Cu at (160.0, 94.2)
- added kibuzzard-676F4471: G***, kibuzzard-676F4471, F.Cu at (175.0, 99.5)
- added kibuzzard-676F4476: G***, kibuzzard-676F4476, F.Cu at (145.5, 99.5)
- moved CN2 0.25 mm to (170.0, 125.8)
- moved CN3 0.25 mm to (170.0, 94.2)
- moved CN4 0.25 mm to (150.0, 94.2)
- moved CN5 0.25 mm to (150.0, 125.8)
- moved JP1 0.05 mm to (164.9, 130.2)
Routing:
- net /Block Diagram/5V: track 20.6 -> 8.56 mm
- net GND: vias 0 -> 52
- added copper zone on F.Cu, net /Block Diagram/5V
Other:
- outline, holes or cut-outs redrawn

Commit message: Updates and fixes
Parts:
- moved kibuzzard-676F3F6C 0.50 mm to (176.5, 116.2)
- moved kibuzzard-676F3F74 0.50 mm to (143.5, 116.2)
Routing:
- net GND: vias 52 -> 51
Other:
- board text added: ">"

Commit message: Fix for 40mm
Parts:
- added kibuzzard-678BDE27: G***, kibuzzard-678BDE27, F.Cu at (160.0, 125.8)
- moved kibuzzard-676F3F6C 1.60 mm to (177.5, 117.5)
- moved kibuzzard-676F3F74 1.46 mm to (142.8, 117.5)
- renumbered CN3 to CN1, CN1 to CN2, CN2 to CN3, CN6 to CN5, CN5 to CN6
Routing:
- net GND: vias 51 -> 68
Other:
- board size 40 x 44 mm -> 44 x 44 mm
- board text added: "^"
- board text removed: ">"
