File: AstraControlPowerPCB/AstraControlPower.kicad_pcb (KiCad board)
At the start: 4 copper layers, 44 x 44 mm, 42 parts, among them CN1 WJ124_5P, CN2 WJ124_5P, CN3 WJ124_5P, CN4 WJ124_5P, CN5 WJ124_5P, CN6 WJ124_5P

Commit message: Slimmer design temp
Parts:
- added H1: MountingHole_Pad, MountingHole:MountingHole_5.3mm_M5_Pad_Via, F.Cu at (170.0, 76.0)
- added H2: MountingHole_Pad, MountingHole:MountingHole_5.3mm_M5_Pad_Via, F.Cu at (150.0, 76.0)
- added H3: MountingHole_Pad, MountingHole:MountingHole_5.3mm_M5_Pad_Via, F.Cu at (150.0, 144.0)
- added H4: MountingHole_Pad, MountingHole:MountingHole_5.3mm_M5_Pad_Via, F.Cu at (170.0, 144.0)
- moved kibuzzard-676F3FB0 96.2 mm to (230.8, 162.0)
- moved kibuzzard-676F4476 96.2 mm to (232.2, 141.0)
- moved kibuzzard-676F3F74 95.5 mm to (232.2, 150.8)
- moved kibuzzard-676F3DF6 82.5 mm to (214.2, 133.0)
- moved kibuzzard-676F3E04 82.5 mm to (218.0, 133.0)
- moved kibuzzard-676F3E0A 82.5 mm to (221.8, 133.0)
- moved kibuzzard-676F3E29 82.5 mm to (225.8, 133.0)
- moved kibuzzard-676F3E9C 82.5 mm to (245.8, 133.0)
- moved kibuzzard-676F3EA0 82.5 mm to (242.0, 133.0)
- moved kibuzzard-676F3EA4 82.5 mm to (238.0, 133.0)
- moved kibuzzard-676F3EA7 82.5 mm to (234.2, 133.0)
- moved kibuzzard-676F4065 82.2 mm to (214.5, 155.8)
- moved kibuzzard-676F39FE 78.4 mm to (226.5, 128.0)
- moved kibuzzard-676F3A03 78.4 mm to (226.5, 120.2)
- moved kibuzzard-676F3A03 78.4 mm to (249.0, 120.2)
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Connections:
- CN2 pad 1: /Block Diagram/5V -> /Block Diagram/VIN
- CN2 pad 2: /Block Diagram/VIN -> /Block Diagram/5V
- CN4 pad 2: /Block Diagram/RS485+ -> /Block Diagram/RS485-
- CN4 pad 3: /Block Diagram/RS485- -> /Block Diagram/RS485+
- CN5 pad 4: /Block Diagram/VIN -> /Block Diagram/5V
- CN5 pad 5: /Block Diagram/5V -> /Block Diagram/VIN
Routing:
- net /Block Diagram/VIN_SW: track 0.00 -> 10.6 mm
- net /Block Diagram/RS485+: track 27.7 -> 32.1 mm
- net /Block Diagram/VIN: track 25.3 -> 27.9 mm
- net /Block Diagram/LED: track 4.26 -> 6.51 mm
- net GND: track 0.00 -> 0.04 mm, vias 68 -> 0
- removed copper zone on F.Cu, net /Block Diagram/5V
- removed copper zone on F.Cu, net /Block Diagram/VIN
- removed copper zone on B.Cu, net /Block Diagram/VIN_SW
Other:
- board size 44 x 44 mm -> 32 x 80 mm
- board text removed: "^"
