File: AstraControlPowerPCB/block_diagram.kicad_sch (KiCad schematic)
At the start: 1 part, among them CN1 WJ124_5P

Commit message: Finished layout
Parts:
- added CN2, CN3, CN4, CN5: WJ124_5P, LiveAstra:CN_SCREW_TERMINAL_WJ124_4P-P3.81_KF124-4P, symbol LiveAstra:CN_SCREW_TERMINAL_WJ124_4P_15A
- added CN6: WJ124_5P, LiveAstra:CN_SCREW_TERMINAL_WJ124_5P-P3.81_KF124-5P, symbol LiveAstra:CN_SCREW_TERMINAL_WJ124_5P_15A
- added JP1: JP_SolderJumper_2_Bridged, Jumper:SolderJumper-2_P1.3mm_Bridged_RoundedPad1.0x1.5mm, symbol LiveAstra:JP_SolderJumper_2_Bridged
- added SW1: SW_SPST_LED, symbol Switch:SW_SPST_LED
- CN1: footprint LiveAstra:CN_SCREW_TERMINAL_WJ124_5P-P3.81_KF124-3.81-5P -> LiveAstra:CN_SCREW_TERMINAL_WJ124_5P-P3.81_KF124-5P
Connections:
- net GND: now also CN2.3 (Pin_3), CN3.2 (Pin_2), CN3.3 (Pin_3), CN4.1 (Pin_1), CN5.2 (Pin_2), CN5.3 (Pin_3), CN6.3 (Pin_3); no longer CN1.1 (Pin_1), CN1.2 (Pin_2), CN1.4 (Pin_4), CN1.5 (Pin_5)
- new net 5V: CN1.1 (Pin_1), CN3.1 (Pin_1), CN4.4 (Pin_4), CN5.1 (Pin_1), CN5.4 (Pin_4), CN6.5 (Pin_5)
- new net LED: CN2.4 (Pin_4), JP1.2 (B)
- new net RS485+: CN1.4 (Pin_4), CN4.2 (Pin_2), CN6.2 (Pin_2)
- new net RS485-: CN1.5 (Pin_5), CN4.3 (Pin_3), CN6.1 (Pin_1)
- new net VIN: CN1.2 (Pin_2), CN2.1 (Pin_1), CN6.4 (Pin_4), JP1.1 (A)
- new net VIN_SW: CN2.2 (Pin_2), CN3.4 (Pin_4)
Other:
- note added: "A Negative White B Positve Blue"
- note added: "Extra 5V Out"
- note added: "Input"
- note added: "Output"
- note added: "To Control Board"
- note added: "To LED Switch"
- note added: "VIN to 5V Converter"

Commit message: Updates and fixes
Other:
- moved on the sheet: CN1, CN2, CN3, CN4, CN5, CN6, JP1, SW1

Commit message: Fix for 40mm
Parts:
- renumbered CN3 to CN1, CN1 to CN2, CN2 to CN3, CN6 to CN5, CN5 to CN6
Changed lines of the file:
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@@
 		(dnp no)
 		(fields_autoplaced yes)
-		(property "Reference" "#PWR03"
+		(property "Reference" "#PWR01"
 			(at 83.82 138.43 0)
 			(effects
@@
 			(project "AstraControlPower"
 				(path "/7280d034-363a-4c4e-8eb5-3b1e5eac524c/274ad830-1c1d-406b-a66e-b0330f7ac6d2"
-					(reference "#PWR03")
+					(reference "#PWR01")
 					(unit 1)
 				)
@@
 		(dnp no)
 		(fields_autoplaced yes)
-		(property "Reference" "#PWR05"
+		(property "Reference" "#PWR09"
 			(at 185.42 135.89 0)
 			(effects
@@
 			(project "AstraControlPower"
 				(path "/7280d034-363a-4c4e-8eb5-3b1e5eac524c/274ad830-1c1d-406b-a66e-b0330f7ac6d2"
-					(reference "#PWR05")
+					(reference "#PWR09")
 					(unit 1)
 				)
@@
 		(dnp no)
 		(fields_autoplaced yes)
-		(property "Reference" "CN3"
+		(property "Reference" "CN1"
 			(at 104.14 123.1899 0)
 			(effects
@@
 			(project "AstraControlPower"
 				(path "/7280d034-363a-4c4e-8eb5-3b1e5eac524c/274ad830-1c1d-406b-a66e-b0330f7ac6d2"
-					(reference "CN3")
+					(reference "CN1")
 					(unit 1)
 				)
@@
 		(dnp no)
 		(fields_autoplaced yes)
-		(property "Reference" "CN6"
+		(property "Reference" "CN5"
 			(at 180.34 48.2599 0)
 			(effects
@@
 			(project ""
 				(path "/7280d034-363a-4c4e-8eb5-3b1e5eac524c/274ad830-1c1d-406b-a66e-b0330f7ac6d2"
-					(reference "CN6")
+					(reference "CN5")
 					(unit 1)
 				)
@@
 		(dnp no)
 		(fields_autoplaced yes)
-		(property "Reference" "#PWR02"
+		(property "Reference" "#PWR04"
 			(at 134.62 95.25 0)
 			(effects
@@
 			(project "AstraControlPower"
 				(path "/7280d034-363a-4c4e-8eb5-3b1e5eac524c/274ad830-1c1d-406b-a66e-b0330f7ac6d2"
-					(reference "#PWR02")
+					(reference "#PWR04")
 					(unit 1)
 				)
@@
 		(dnp no)
 		(fields_autoplaced yes)
-		(property "Reference" "#PWR01"
+		(property "Reference" "#PWR02"
 			(at 109.22 59.69 0)
 			(effects
@@
 			(project "AstraControlPower"
 				(path "/7280d034-363a-4c4e-8eb5-3b1e5eac524c/274ad830-1c1d-406b-a66e-b0330f7ac6d2"
-					(reference "#PWR01")
+					(reference "#PWR02")
 					(unit 1)
 				)
@@
 		(dnp no)
 		(fields_autoplaced yes)
-		(property "Reference" "CN1"
+		(property "Reference" "CN2"
 			(at 129.54 48.2599 0)
 			(effects
@@
 			(project ""
 				(path "/7280d034-363a-4c4e-8eb5-3b1e5eac524c/274ad830-1c1d-406b-a66e-b0330f7ac6d2"
-					(reference "CN1")
+					(reference "CN2")
 					(unit 1)
 				)
@@
 		(dnp no)
 		(fields_autoplaced yes)
-		(property "Reference" "CN2"
+		(property "Reference" "CN3"
 			(at 154.94 82.5499 0)
 			(effects
@@
 			(project ""
 				(path "/7280d034-363a-4c4e-8eb5-3b1e5eac524c/274ad830-1c1d-406b-a66e-b0330f7ac6d2"
-					(reference "CN2")
+					(reference "CN3")
 					(unit 1)
 				)
@@
 		(dnp no)
 		(fields_autoplaced yes)
-		(property "Reference" "CN5"
+		(property "Reference" "CN6"
 			(at 205.74 123.1899 0)
 			(effects
@@
 			(project "AstraControlPower"
 				(path "/7280d034-363a-4c4e-8eb5-3b1e5eac524c/274ad830-1c1d-406b-a66e-b0330f7ac6d2"
-					(reference "CN5")
+					(reference "CN6")
 					(unit 1)
 				)
@@
 		(dnp no)
 		(fields_autoplaced yes)
-		(property "Reference" "#PWR04"
+		(property "Reference" "#PWR05"
 			(at 134.62 130.81 0)
 			(effects
@@
 			(project "AstraControlPower"
 				(path "/7280d034-363a-4c4e-8eb5-3b1e5eac524c/274ad830-1c1d-406b-a66e-b0330f7ac6d2"
-					(reference "#PWR04")
-					(unit 1)
-				)
+					(reference "#PWR05")
+					(unit 1)
+				)

Commit message: Slimmer design temp
Parts:
- added H1, H2, H3, H4: MountingHole_Pad, MountingHole:MountingHole_5.3mm_M5_Pad_Via, symbol LiveAstra:MountingHole_Pad
Connections:
- net 5V: now also CN2.2 (Pin_2), CN5.4 (Pin_4); no longer CN2.1 (Pin_1), CN5.5 (Pin_5)
- net GND: now also H1.1, H2.1, H3.1, H4.1
- net RS485+: now also CN4.3 (Pin_3); no longer CN4.2 (Pin_2)
- net RS485-: now also CN4.2 (Pin_2); no longer CN4.3 (Pin_3)
- net VIN: now also CN2.1 (Pin_1), CN5.5 (Pin_5); no longer CN2.2 (Pin_2), CN5.4 (Pin_4)
